File: pcb_files/mini/Front_panel_owon_ver_mini.brd (EAGLE design)
At the start: 49 x 99 mm, 18 parts, among them M1 ARDUINO-NANO-3.0, SW1 ROTARTY_ENCODER, SW2 TACTILE-SWITCH-PTH, SW3 TACTILE-SWITCH-PTH, SW4 TACTILE-SWITCH-PTH

Commit message: retoques, mejoras y agregados
Parts:
- added U$2: (no value), adafruit:OSHWLOGO_TOP_0.2
- added U$3: (no value), adafruit:OSHWLOGO_TOL_0.2
- moved SW1 0.38 mm to (25.0, 73.0)
- moved SW4 0.38 mm to (25.0, 10.0)
- moved SW2 0.37 mm to (25.0, 50.0)
- moved SW3 0.36 mm to (25.0, 30.0)
- moved LED3 0.36 mm to (38.0, 94.0)
- moved LED2 0.36 mm to (25.0, 94.0)
- moved LED1 0.35 mm to (12.0, 94.0)
- renumbered M1 to U1
Routing:
- net D2: track 55.1 -> 56.5 mm
- net 5V: track 102.7 -> 101.6 mm
- net D4: track 52.0 -> 52.8 mm
Other:
- outline, holes or cut-outs redrawn
- board text added: "FRONT PANEL OWON"
- board text removed: "DOCK OWON"
